File: 24-5_buck.kicad_sch (KiCad schematic)
At the start: 8 parts, among them IC4 LMR51610YDBVR

Commit message: Finalize KiCad PCB sources for 5-piece test build
Commit the completed Open Vettam 15CCT KiCad source design files prepared for the initial five-piece production test run.

Included files are limited to the schematic hierarchy, PCB layouts, KiCad project files, and the LED MCPCB design-rules file. Generated BOM exports, fabrication output archives, freerouting/temp files, logs, backups, images, netlists, and Altium import artifacts are intentionally left unstaged.

Updated main controller board sources:

- open_vettam_15CCT.kicad_sch

- open_vettam_15CCT.kicad_pcb

- open_vettam_15CCT.kicad_pro

- 24v_Input.kicad_sch

- 24-5_buck.kicad_sch

- MCU.kicad_sch

- cc_driver.kicad_sch

Updated LED MCPCB sources:

- led_mcpcb/led_mcpcb.kicad_sch

- led_mcpcb/led_mcpcb.kicad_pcb

- led_mcpcb/led_mcpcb.kicad_pro

- led_mcpcb/led_mcpcb.kicad_dru

- led_mcpcb/CW-5000.kicad_sch

- led_mcpcb/WW-3000.kicad_sch

- led_mcpcb/digital_temp.kicad_sch
Parts:
- C18, C19: value 0.1ÂµF 50V -> 0.1µF 50V
- C20: value 2.2ÂµF 50V -> 2.2µF 50V
- C21: value 10ÂµF 16V -> 10µF 16V
- L3: value 10ÂµH -> 10µH; Mouser Part Number (none) -> 652-SRP5030HMT-100M
Changed lines of the file:
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@@
 			)
 		)
-		(property "Value" "0.1ÂµF 50V"
+		(property "Value" "0.1µF 50V"
 			(at 151.13 114.2999 90)
 			(show_name no)
@@
 			)
 		)
-		(property "Value" "10ÂµH"
+		(property "Value" "10µH"
 			(at 168.91 80.01 0)
 			(show_name no)
@@
 			)
 		)
-		(property "Mouser Part Number" ""
+		(property "Mouser Part Number" "652-SRP5030HMT-100M"
 			(at 175.26 780.01 0)
 			(hide yes)
@@
 			)
 		)
-		(property "Value" "2.2ÂµF 50V"
+		(property "Value" "2.2µF 50V"
 			(at 167.64 114.2999 90)
 			(show_name no)
@@
 			)
 		)
-		(property "Value" "10ÂµF 16V"
+		(property "Value" "10µF 16V"
 			(at 213.36 115.5699 90)
 			(show_name no)
@@
 			)
 		)
-		(property "Value" "0.1ÂµF 50V"
+		(property "Value" "0.1µF 50V"
 			(at 139.7 78.74 0)
 			(show_name no)
