File: 24v_Input.kicad_sch (KiCad schematic)
At the start: 9 parts, among them J1 24VIN, Q1 SQJ457EP-T1_BE3

Commit message: Finalize KiCad PCB sources for 5-piece test build
Commit the completed Open Vettam 15CCT KiCad source design files prepared for the initial five-piece production test run.

Included files are limited to the schematic hierarchy, PCB layouts, KiCad project files, and the LED MCPCB design-rules file. Generated BOM exports, fabrication output archives, freerouting/temp files, logs, backups, images, netlists, and Altium import artifacts are intentionally left unstaged.

Updated main controller board sources:

- open_vettam_15CCT.kicad_sch

- open_vettam_15CCT.kicad_pcb

- open_vettam_15CCT.kicad_pro

- 24v_Input.kicad_sch

- 24-5_buck.kicad_sch

- MCU.kicad_sch

- cc_driver.kicad_sch

Updated LED MCPCB sources:

- led_mcpcb/led_mcpcb.kicad_sch

- led_mcpcb/led_mcpcb.kicad_pcb

- led_mcpcb/led_mcpcb.kicad_pro

- led_mcpcb/led_mcpcb.kicad_dru

- led_mcpcb/CW-5000.kicad_sch

- led_mcpcb/WW-3000.kicad_sch

- led_mcpcb/digital_temp.kicad_sch
Parts:
- C22: value 47ÂµF 50V -> 47µF 50V
Changed lines of the file:
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@@
 			)
 		)
-		(property "Value" "47ÂµF 50V"
+		(property "Value" "47µF 50V"
 			(at 232.41 99.0599 90)
 			(show_name no)
