File: MCU.kicad_sch (KiCad schematic)
At the start: 12 parts, among them IC1 ESP32-C6-MINI-1-N4, J2 DEBUG, J5 TEMP_IN

Commit message: Finalize KiCad PCB sources for 5-piece test build
Commit the completed Open Vettam 15CCT KiCad source design files prepared for the initial five-piece production test run.

Included files are limited to the schematic hierarchy, PCB layouts, KiCad project files, and the LED MCPCB design-rules file. Generated BOM exports, fabrication output archives, freerouting/temp files, logs, backups, images, netlists, and Altium import artifacts are intentionally left unstaged.

Updated main controller board sources:

- open_vettam_15CCT.kicad_sch

- open_vettam_15CCT.kicad_pcb

- open_vettam_15CCT.kicad_pro

- 24v_Input.kicad_sch

- 24-5_buck.kicad_sch

- MCU.kicad_sch

- cc_driver.kicad_sch

Updated LED MCPCB sources:

- led_mcpcb/led_mcpcb.kicad_sch

- led_mcpcb/led_mcpcb.kicad_pcb

- led_mcpcb/led_mcpcb.kicad_pro

- led_mcpcb/led_mcpcb.kicad_dru

- led_mcpcb/CW-5000.kicad_sch

- led_mcpcb/WW-3000.kicad_sch

- led_mcpcb/digital_temp.kicad_sch
Parts:
- R3, R5: Manufacturer_Name (none) -> Yageo Group; Manufacturer_Part_Number (none) -> RC0603FR-0710KL; Mouser Part Number (none) -> 603-RC0603FR-0710KL
Connections:
- net BOOT: now reaches IC1.23 (IO9), J2.6 (Pin_6)
Changed lines of the file:
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@@
-		)
-	)
-	(label ""
-		(at 119.38 123.19 0)
-		(effects
-			(font
-				(size 1.27 1.27)
-			)
-			(justify left bottom)
 		)
 	)
@@
 	)
 	(label "BOOT"
-		(at 114.3 123.19 0)
+		(at 114.3 123.19 180)
 		(effects
 			(font
 				(size 1.27 1.27)
 			)
-			(justify left bottom)
+			(justify right bottom)
 		)
 	)
@@
 			)
 		)
-		(property "Datasheet" ""
+		(property "Datasheet" "https://www.yageo.com/upload/media/product/productsearch/datasheet/rchip/PYu-RC_Group_51_RoHS_L_12.pdf"
 			(at 99.06 114.3 0)
 			(hide yes)
@@
 			)
 		)
+		(property "Manufacturer_Name" "Yageo Group" (at 99.06 114.3 0) (hide yes) (effects (font (size 1.27 1.27))))
+		(property "Manufacturer_Part_Number" "RC0603FR-0710KL" (at 99.06 114.3 0) (hide yes) (effects (font (size 1.27 1.27))))
+		(property "Mouser Part Number" "603-RC0603FR-0710KL" (at 99.06 114.3 0) (hide yes) (effects (font (size 1.27 1.27))))
 		(pin "2"
 		)
@@
 			)
 		)
-		(property "Datasheet" ""
+		(property "Datasheet" "https://www.yageo.com/upload/media/product/productsearch/datasheet/rchip/PYu-RC_Group_51_RoHS_L_12.pdf"
 			(at 83.82 77.47 0)
 			(hide yes)
@@
 			)
 		)
+		(property "Manufacturer_Name" "Yageo Group" (at 83.82 77.47 0) (hide yes) (effects (font (size 1.27 1.27))))
+		(property "Manufacturer_Part_Number" "RC0603FR-0710KL" (at 83.82 77.47 0) (hide yes) (effects (font (size 1.27 1.27))))
+		(property "Mouser Part Number" "603-RC0603FR-0710KL" (at 83.82 77.47 0) (hide yes) (effects (font (size 1.27 1.27))))
 		(pin "2"
 		)
