File: led_mcpcb/CW-5000.kicad_sch (KiCad schematic)
At the start: 50 parts

Commit message: Finalize KiCad PCB sources for 5-piece test build
Commit the completed Open Vettam 15CCT KiCad source design files prepared for the initial five-piece production test run.

Included files are limited to the schematic hierarchy, PCB layouts, KiCad project files, and the LED MCPCB design-rules file. Generated BOM exports, fabrication output archives, freerouting/temp files, logs, backups, images, netlists, and Altium import artifacts are intentionally left unstaged.

Updated main controller board sources:

- open_vettam_15CCT.kicad_sch

- open_vettam_15CCT.kicad_pcb

- open_vettam_15CCT.kicad_pro

- 24v_Input.kicad_sch

- 24-5_buck.kicad_sch

- MCU.kicad_sch

- cc_driver.kicad_sch

Updated LED MCPCB sources:

- led_mcpcb/led_mcpcb.kicad_sch

- led_mcpcb/led_mcpcb.kicad_pcb

- led_mcpcb/led_mcpcb.kicad_pro

- led_mcpcb/led_mcpcb.kicad_dru

- led_mcpcb/CW-5000.kicad_sch

- led_mcpcb/WW-3000.kicad_sch

- led_mcpcb/digital_temp.kicad_sch
Parts:
- removed CW+, CW-: PAD, TestPoint:TestPoint_Pad_2.5x2.5mm, symbol Connector:TestPoint
- added J1: CW+, Connector_Wire:SolderWirePad_1x01_SMD_5x10mm, symbol Connector_Generic:Conn_01x01
- added J2: CW-, Connector_Wire:SolderWirePad_1x01_SMD_5x10mm, symbol Connector_Generic:Conn_01x01
- renumbered LED9 to LED10, LED10 to LED11, LED11 to LED12, LED12 to LED13, LED56 to LED14, LED13 to LED15, LED14 to LED16, LED15 to LED17, LED16 to LED18, LED17 to LED19, LED18 to LED20, LED57 to LED21, LED19 to LED22, LED20 to LED23, LED21 to LED24, LED22 to LED25, LED23 to LED26, LED24 to LED27, LED58 to LED28, LED49 to LED29, LED50 to LED30, LED51 to LED31, LED52 to LED32, LED53 to LED33, LED54 to LED34, LED63 to LED35, LED64 to LED36, LED65 to LED37, LED66 to LED38, LED67 to LED39, LED68 to LED40, LED69 to LED41, LED70 to LED42, LED55 to LED7, LED7 to LED8, LED8 to LED9, R11 to R1, R12 to R2, R13 to R3, R14 to R4, R15 to R5, R16 to R6
Connections:
- net GND: now also J2.1 (Pin_1)
- net vcc: no longer names the net of R1.2, R2.2, R3.2, R4.2, R5.2, R6.2
- net vcc: now also J1.1 (Pin_1)
