File: led_mcpcb/WW-3000.kicad_sch (KiCad schematic)
At the start: 50 parts

Commit message: Finalize KiCad PCB sources for 5-piece test build
Commit the completed Open Vettam 15CCT KiCad source design files prepared for the initial five-piece production test run.

Included files are limited to the schematic hierarchy, PCB layouts, KiCad project files, and the LED MCPCB design-rules file. Generated BOM exports, fabrication output archives, freerouting/temp files, logs, backups, images, netlists, and Altium import artifacts are intentionally left unstaged.

Updated main controller board sources:

- open_vettam_15CCT.kicad_sch

- open_vettam_15CCT.kicad_pcb

- open_vettam_15CCT.kicad_pro

- 24v_Input.kicad_sch

- 24-5_buck.kicad_sch

- MCU.kicad_sch

- cc_driver.kicad_sch

Updated LED MCPCB sources:

- led_mcpcb/led_mcpcb.kicad_sch

- led_mcpcb/led_mcpcb.kicad_pcb

- led_mcpcb/led_mcpcb.kicad_pro

- led_mcpcb/led_mcpcb.kicad_dru

- led_mcpcb/CW-5000.kicad_sch

- led_mcpcb/WW-3000.kicad_sch

- led_mcpcb/digital_temp.kicad_sch
Parts:
- removed WW+, WW-: PAD, TestPoint:TestPoint_Pad_2.5x2.5mm, symbol Connector:TestPoint
- added J3: WW+, Connector_Wire:SolderWirePad_1x01_SMD_5x10mm, symbol Connector_Generic:Conn_01x01
- added J4: WW-, Connector_Wire:SolderWirePad_1x01_SMD_5x10mm, symbol Connector_Generic:Conn_01x01
- renumbered LED25 to LED43, LED26 to LED44, LED27 to LED45, LED28 to LED46, LED29 to LED47, LED30 to LED48, LED59 to LED49, LED31 to LED50, LED32 to LED51, LED33 to LED52, LED34 to LED53, LED35 to LED54, LED36 to LED55, LED60 to LED56, LED37 to LED57, LED38 to LED58, LED39 to LED59, LED40 to LED60, LED41 to LED61, LED42 to LED62, LED61 to LED63, LED43 to LED64, LED44 to LED65, LED45 to LED66, LED46 to LED67, LED47 to LED68, LED48 to LED69, LED62 to LED70, R8 to R10, R9 to R11, R10 to R12, R5 to R7, R6 to R8, R7 to R9
Connections:
- net GND: now also J4.1 (Pin_1)
- net vcc: no longer names the net of R10.2, R11.2, R12.2, R7.2, R8.2, R9.2
- net vcc: now also J3.1 (Pin_1)
